File: hw/controller/controller.brd (EAGLE design)
At the start: 45 x 45 mm, 93 parts, among them J1 JST-PH3SMT_VERT, J2 JST-PH3SMT_VERT, M3 PAD24AWG_PAD, Q1 TPN1R603PL, Q2 TPN1R603PL, Q3 TPN1R603PL, Q4 TPN1R603PL, Q5 TPN1R603PL, Q6 TPN1R603PL, U1 STM32F4R_64PIN, U2 DRV8323RS, U3 AS5147, U4 MAX13431E, U5 MAX13433EETD+T, X1 8.0MHz

Commit message: More work on controller board
Parts:
- moved R12 0.30 mm to (36.7, 5.90)
Connections:
- net GND: now also U1.2
Routing:
- net GND: track 74.7 -> 76.3 mm, vias 32 -> 33
Changed lines of the file:
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@@
 <attribute name="NAME" x="27.5" y="33.5" size="0.6096" layer="25" font="vector" ratio="10" rot="R180"/>
 </element>
-<element name="R12" library="mfpassives" package="R0402" value="47k NTC" x="36.4" y="5.9" smashed="yes" rot="R90">
-<attribute name="HOUSEPART" value="" x="36.4" y="5.9" size="0.8" layer="27" rot="R90" display="off"/>
-<attribute name="TOLERANCE" value="" x="36.4" y="5.9" size="0.8" layer="27" rot="R90" display="off"/>
-<attribute name="MPN" value="NCP15WB473F03RC" x="36.4" y="5.9" size="0.8" layer="27" rot="R90" display="off"/>
-<attribute name="POPULATE" value="1" x="36.4" y="5.9" size="0.8" layer="27" rot="R90" display="off"/>
-<attribute name="VOLTAGE" value="" x="36.4" y="5.9" size="0.8" layer="27" rot="R90" display="off"/>
-<attribute name="MF" value="Murata" x="36.4" y="5.9" size="0.8" layer="27" rot="R90" display="off"/>
-<attribute name="URL" value="" x="36.4" y="5.9" size="0.8" layer="27" rot="R90" display="off"/>
-<attribute name="WATTAGE" value="" x="36.4" y="5.9" size="0.8" layer="27" rot="R90" display="off"/>
-<attribute name="NAME" x="37.8" y="5.5" size="0.6096" layer="25" font="vector" ratio="10" rot="R90"/>
+<element name="R12" library="mfpassives" package="R0402" value="47k NTC" x="36.7" y="5.9" smashed="yes" rot="R90">
+<attribute name="HOUSEPART" value="" x="36.7" y="5.9" size="0.8" layer="27" rot="R90" display="off"/>
+<attribute name="TOLERANCE" value="" x="36.7" y="5.9" size="0.8" layer="27" rot="R90" display="off"/>
+<attribute name="MPN" value="NCP15WB473F03RC" x="36.7" y="5.9" size="0.8" layer="27" rot="R90" display="off"/>
+<attribute name="POPULATE" value="1" x="36.7" y="5.9" size="0.8" layer="27" rot="R90" display="off"/>
+<attribute name="VOLTAGE" value="" x="36.7" y="5.9" size="0.8" layer="27" rot="R90" display="off"/>
+<attribute name="MF" value="Murata" x="36.7" y="5.9" size="0.8" layer="27" rot="R90" display="off"/>
+<attribute name="URL" value="" x="36.7" y="5.9" size="0.8" layer="27" rot="R90" display="off"/>
+<attribute name="WATTAGE" value="" x="36.7" y="5.9" size="0.8" layer="27" rot="R90" display="off"/>
+<attribute name="NAME" x="38.1" y="5.5" size="0.6096" layer="25" font="vector" ratio="10" rot="R90"/>
 </element>
 <element name="R13" library="mfpassives" package="R0402" value="10k 1%" x="36.7" y="8.4" smashed="yes" rot="R90">
@@
 <wire x1="12" y1="36.7" x2="12" y2="37.47" width="0.254" layer="1"/>
 <wire x1="12" y1="37.47" x2="11.97" y2="37.5" width="0.254" layer="1"/>
-<via x="12.4" y="35.4" extent="1-16" drill="0.4"/>
+<via x="12.4" y="35.5" extent="1-16" drill="0.4"/>
 <wire x1="10.93" y1="35.47" x2="12.13" y2="35.47" width="0.254" layer="1"/>
-<wire x1="12.13" y1="35.47" x2="12.4" y2="35.4" width="0.254" layer="1"/>
+<wire x1="12.13" y1="35.47" x2="12.4" y2="35.5" width="0.254" layer="1"/>
 <via x="27.3" y="28" extent="1-16" drill="0.4"/>
 <wire x1="26.52" y1="28.58" x2="27.22" y2="28.02" width="0.4064" layer="1"/>
@@
 <wire x1="35.8" y1="17.2" x2="35.8" y2="6" width="0.127" layer="1"/>
 <wire x1="35" y1="18" x2="35.8" y2="17.2" width="0.127" layer="1"/>
-<wire x1="36.4" y1="5.4" x2="36.4" y2="5.35" width="0.127" layer="1"/>
+<wire x1="36.4" y1="5.4" x2="36.7" y2="5.35" width="0.127" layer="1"/>
 <wire x1="35" y1="18" x2="34.9" y2="18" width="0.127" layer="1"/>
 <contactref element="TEMP1" pad="P$1"/>
@@
 <wire x1="13.25" y1="38.7" x2="13.49" y2="38.94" width="0.3048" layer="1"/>
 <contactref element="DGND" pad="P$1"/>
+<contactref element="U1" pad="2"/>
+<via x="12.39" y="34.59" extent="1-16" drill="0.4"/>
+<wire x1="10.93" y1="34.97" x2="12.01" y2="34.97" width="0.127" layer="1"/>
+<wire x1="12.01" y1="34.97" x2="12.39" y2="34.59" width="0.127" layer="1"/>
 </signal>
 <signal name="DBG_Y">
@@
 <contactref element="R13" pad="P$1"/>
 <contactref element="U1" pad="10"/>
-<wire x1="36.6" y1="6.8" x2="36.4" y2="6.6" width="0.127" layer="1"/>
-<wire x1="36.6" y1="7.8" x2="36.6" y2="6.8" width="0.127" layer="1"/>
-<wire x1="36.4" y1="6.6" x2="36.4" y2="6.45" width="0.127" layer="1"/>
-<wire x1="36.6" y1="7.8" x2="36.7" y2="7.85" width="0.127" layer="1"/>
+<wire x1="36.7" y1="7.85" x2="36.7" y2="6.45" width="0.127" layer="1"/>
+<wire x1="36.7" y1="7.9" x2="36.7" y2="7.85" width="0.127" layer="1"/>
 <wire x1="37.95" y1="8" x2="36.8" y2="8" width="0.127" layer="1"/>
 <wire x1="38.8" y1="12.8" x2="38.8" y2="8" width="0.127" layer="1"/>
@@
 <contactref element="U1" pad="8"/>
 <wire x1="13" y1="32" x2="11" y2="32" width="0.127" layer="1"/>
-<wire x1="13" y1="36" x2="13" y2="32" width="0.127" layer="1"/>
-<wire x1="11.4" y1="36" x2="13" y2="36" width="0.127" layer="1"/>
-<wire x1="11.4" y1="40.2" x2="11.4" y2="36" width="0.127" layer="1"/>
+<wire x1="13" y1="36.1" x2="13" y2="32" width="0.127" layer="1"/>
+<wire x1="11.4" y1="36.1" x2="13" y2="36.1" width="0.127" layer="1"/>
+<wire x1="11.4" y1="40.2" x2="11.4" y2="36.1" width="0.127" layer="1"/>
 <wire x1="11" y1="32" x2="10.93" y2="31.97" width="0.127" layer="1"/>
 <wire x1="11.4" y1="40.2" x2="12.15" y2="40.4" width="0.127" layer="1"/>

Commit message: Progress on controller r3
Parts:
- added C33, C34, C35, C36, C37, C38: 10uF, mfpassives:C1206
- C14, C15, C16, C17, C18, C19, C20: value 15uF -> 10uF
- R1: device mfpassives:R0603 -> mfpassives:R0402
- moved R5 1.02 mm to (11.7, 40.2)
- moved C30 0.86 mm to (29.3, 34.0)
- moved C31 0.86 mm to (29.3, 32.7)
- moved U5 0.86 mm to (28.7, 36.5)
- moved DTX 0.76 mm to (17.4, 39.0)
- moved R1 0.65 mm to (14.7, 39.4), turned to 270 degrees
- moved DRX 0.60 mm to (16.0, 39.3)
- moved SWD 0.58 mm to (35.8, 35.6)
- moved LNK 0.58 mm to (23.9, 40.6)
- moved SH3 0.41 mm to (33.6, 12.0)
- moved V- 0.14 mm to (4.40, 11.0)
- moved ABS_SCL 0.10 mm to (16.6, 41.5)
- moved ABS_SDA 0.10 mm to (16.6, 43.1)
Connections:
- net GND: now also U1.3; no longer U1.2
- net V+: now also C33.P$1, C34.P$1, C35.P$1, C36.P$1, C37.P$1, C38.P$1
- net V-: now also C33.P$2, C34.P$2, C35.P$2, C36.P$2, C37.P$2, C38.P$2
Routing:
- net VTEMP_FET: track 48.1 -> 60.6 mm
- net I2C_ABS_SDA: track 7.32 -> 10.8 mm, vias 0 -> 1
- net I2C_ABS_SCL: track 5.59 -> 7.70 mm
- net GND: track 76.3 -> 75.1 mm
- net DBG_A: track 9.06 -> 10.2 mm
- net DBG_Z: track 6.14 -> 7.33 mm
- net DBG_Y: track 5.64 -> 6.83 mm
- net DBG_B: track 7.51 -> 8.65 mm
- net +3V3: track 70.6 -> 71.7 mm
- net DEBUG_TX: track 15.4 -> 16.4 mm
- net DEBUG_RX: track 16.9 -> 17.7 mm
- net N$2: track 3.26 -> 2.64 mm
- net VTEMP_MOT: track 14.8 -> 14.3 mm
- net V-: track 17.3 -> 17.8 mm, vias 25 -> 35
- net V+: vias 13 -> 23
Other:
- board text added: "(c) jjp@pobox.com"
- board text added: "2019"
- board text added: "moteus r3"
- board text removed: "(c) jjp@pobox.com 2018"
- board text removed: "moteus r2"
