File: hw/n1/moteus_n1.brd (EAGLE design)
At the start: 46 x 46 mm, 192 parts, among them J1 XT30XT30PW_MALE, J2 XT30XT30PW_MALE, J3 SM06B-GHS-TB(LF)(SN), M1 MOUNT, M2 MOUNT, M3 MOUNT, M4 MOUNT, Q1 TPH1R204PL_VIAS, Q2 TPH1R204PLSOP_ADVANCE_8, Q3 TPH1R204PL_VIAS, Q4 TPH1R204PLSOP_ADVANCE_8, Q5 TPH1R204PL_VIAS, Q6 TPH1R204PLSOP_ADVANCE_8, U1 MAX15062AATA+T, U2 ADP5301ACBZ-4-R7, U3 STM32G474CEU6, U4 TCAN1042HGV, U5 AS5147, U7 DRV8353S, U8 SN65HVD35DR

Commit message: Update the moteus-n1 5V regulator "value" to be MAX15062BATA+T
The MPN attribute was always correct and is canonical, but this makes
confusion less likely.
Parts:
- U1: value MAX15062AATA+T -> MAX15062BATA+T
Changed lines of the file:
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@@
 <attribute name="POPULATE" value="1" x="17.47863125" y="91.92763125" size="1.778" layer="27" rot="R225" display="off"/>
 </element>
-<element name="U1" library="power_dist" package="21-0487A_MXM" value="MAX15062AATA+T" x="41.4" y="10.6" smashed="yes" rot="MR90">
+<element name="U1" library="power_dist" package="21-0487A_MXM" value="MAX15062BATA+T" x="41.4" y="10.6" smashed="yes" rot="MR90">
 <attribute name="BUILT_BY" value="EMA_Jessica" x="49.7" y="10.6" size="1.778" layer="28" rot="MR90" display="off"/>
 <attribute name="COPYRIGHT" value="Copyright (C) 2018 Accelerated Designs. All rights reserved" x="49.7" y="10.6" size="1.778" layer="28" rot="MR90" display="off"/>
