File: hw/mjuart/mjuart.kicad_sch (KiCad schematic)
At the start: 0 parts

Commit message: mjuart: Fix ZH4 pinout to match moteus-r4
Other:
- title: mjuart r1 -> mjuart r2
Changed lines of the file:
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@@
 	(paper "A4")
 	(title_block
-		(title "mjuart r1")
+		(title "mjuart r2")
 		(company "mjbots Robotic Systems, LLC - info@mjbots.com")
 		(comment 1 "Licensed under the Apache 2.0 License")
